File: kicad/gpio-usb/gpio-usb.sch (KiCad schematic (older format))
At the start: 45 parts, among them J1 USB_A, J2 Conn_01x02_Female, J3 Conn_01x04_Female, J4 Conn_01x06_Female, J5 RJ45, Q1 BSS84, SW1 SW_DPST_x2, U1 MCP1703A-3302_SOT223, U2 AT90USB162-16MU, Y1 8Mhz

Commit message: update booster kicad
Parts:
- removed J5: RJ45, symbol Connector:RJ45
Changed lines of the file:
@@
 EESchema Schematic File Version 4
-LIBS:gpio-usb-cache
 EELAYER 30 0
 EELAYER END
@@
 	8055 2185 8860 2185
 Connection ~ 8055 2205
-$Comp
-L Connector:RJ45 J5
-U 1 1 5D6AA968
-P 1450 6580
-F 0 "J5" H 1507 7247 50  0000 C CNN
-F 1 "RJ45" H 1507 7156 50  0000 C CNN
-F 2 "" V 1450 6605 50  0001 C CNN
-F 3 "~" V 1450 6605 50  0001 C CNN
-	1    1450 6580
-	1    0    0    -1
-$EndComp
 $EndSCHEMATC
