File: kicad/sboxnet-modul/sboxnet-modul.sch (KiCad schematic (older format))
At the start: 34 parts, among them J1 Conn_01x03, J2 Conn_01x04, J4 8P8C, J5 8P8C, J6 sboxnet-buchse_2x17, SW1 SW_Push, U1 MCP1703A-3302_SOT223, U2 MCP1703A-5002_SOT223, U3 SN65HVD230, U4 ATxmega32A4U-AU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

Commit message: update booster layout with POWERSO Slug Down Terminal Vias
Parts:
- J6: symbol sboxnet:sboxnet-buchse_02x17 -> sboxnet-modul-rescue:sboxnet-buchse_02x17-sboxnet
Changed lines of the file:
@@
 	8220 3070 8385 3070
 $Comp
-L sboxnet:sboxnet-buchse_02x17 J6
+L sboxnet-modul-rescue:sboxnet-buchse_02x17-sboxnet J6
 U 1 1 5D99F745
 P 8020 2670
