File: kicad/sboxnet-modul/sboxnet-modul.sch (KiCad schematic (older format))
At the start: 34 parts, among them J1 Conn_01x03, J2 Conn_01x04, J4 8P8C, J5 8P8C, J6 sboxnet-buchse_2x17, SW1 SW_Push, U1 MCP1703A-3302_SOT223, U2 MCP1703A-5002_SOT223, U3 SN65HVD230, U4 ATxmega32A4U-AU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

Commit message: correct sboxnet-modul
Parts:
- J2: footprint Connector_PinHeader_2.54mm:PinHeader_1x04_P2.54mm_Vertical_SMD_Pin1Left -> Connector_PinSocket_2.54mm:PinSocket_1x04_P2.54mm_Vertical
Changed lines of the file:
@@
 F 0 "J2" V 2494 3097 50  0000 R CNN
 F 1 "Conn_01x04" V 2403 3097 50  0000 R CNN
-F 2 "Connector_PinHeader_2.54mm:PinHeader_1x04_P2.54mm_Vertical_SMD_Pin1Left" H 2530 3385 50  0001 C CNN
+F 2 "Connector_PinSocket_2.54mm:PinSocket_1x04_P2.54mm_Vertical" H 2530 3385 50  0001 C CNN
 F 3 "~" H 2530 3385 50  0001 C CNN
 	1    2530 3385
