File: kicad/sboxnet-booster/_autosave-sboxnet-booster.sch (KiCad schematic (older format))
At the start: 52 parts, among them J1 sboxnet-stecker_02x17, J3 Conn_01x02_Male, J4 Conn_01x02_Male, J5 Screw_Terminal_01x04, J6 Screw_Terminal_01x04, J7 Power von externen 15V/4A Net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, SW1 Öffner, U1 L6206PSO-sboxnet, U2 L78L12_SOT89

Commit message: PSO backplane
Parts:
- J7: value Power von externen 15V/4A Netzteil -> Power von externen 15V/4A Netzteil DS_NRJ4HF
Changed lines of the file:
@@
 P 7275 1695
 F 0 "J7" H 7095 1678 50  0000 R CNN
-F 1 "Power von externen 15V/4A Netzteil " H 7095 1769 50  0000 R CNN
+F 1 "Power von externen 15V/4A Netzteil  DS_NRJ4HF" H 7095 1769 50  0000 R CNN
 F 2 "Connector_Audio:Jack_6.35mm_Neutrik_NRJ4HF_Horizontal" H 7275 1695 50  0001 C CNN
 F 3 "~" H 7275 1695 50  0001 C CNN
@@
 	1800 4840 1850 4840
 $Comp
+L Diode:1N4148WS D8
+U 1 1 5F1F6AFD
+P 4315 2300
+F 0 "D8" V 4361 2220 50  0000 R CNN
+F 1 "1N4148WS" V 4270 2220 50  0000 R CNN
+F 2 "Diode_SMD:D_SOD-323" H 4315 2125 50  0001 C CNN
+F 3 "https://www.vishay.com/docs/85751/1n4148ws.pdf" H 4315 2300 50  0001 C CNN
+	1    4315 2300
+	0    -1   -1   0
+$EndComp
+Wire Wire Line
+	4315 2450 4315 2470
+Wire Wire Line
+	4315 2470 4660 2470
+Wire Wire Line
+	4660 2470 4660 2480
+Connection ~ 4315 2470
+Wire Wire Line
+	4315 2470 4315 2490
+$Comp
+L Diode:BAR42FILM D5
+U 1 1 5F0E2174
+P 3410 3442
+F 0 "D5" H 3410 3723 50  0000 C CNN
+F 1 "BAR42FILM" H 3410 3632 50  0000 C CNN
+F 2 "Package_TO_SOT_SMD:SOT-23" H 3410 3267 50  0001 C CNN
+F 3 "www.st.com/resource/en/datasheet/bar42.pdf" H 3410 3442 50  0001 C CNN
+	1    3410 3442
+	1    0    0    -1
+$EndComp
+Text GLabel 3836 3438 2    50   Input ~ 0
+EN
+Wire Wire Line
+	3834 3436 3836 3438
+Wire Wire Line
+	2480 3440 2538 3440
+Wire Wire Line
+	3260 3440 3260 3442
+Connection ~ 2538 3440
+Wire Wire Line
+	3572 3436 3572 3442
+Wire Wire Line
+	3572 3442 3560 3442
+Wire Wire Line
+	3620 3436 3834 3436
+Wire Wire Line
+	3572 3436 3620 3436
+Connection ~ 3620 3436
+$Comp
+L Device:R R9
+U 1 1 5DBEDE1B
+P 3620 3586
+F 0 "R9" H 3550 3540 50  0000 R CNN
+F 1 "2k" H 3550 3631 50  0000 R CNN
+F 2 "Resistor_SMD:R_1206_3216Metric" V 3550 3586 50  0001 C CNN
+F 3 "~" H 3620 3586 50  0001 C CNN
+	1    3620 3586
+	-1   0    0    1
+$EndComp
+$Comp
+L Diode:BAR42FILM D6
+U 1 1 5F139EE6
+P 3618 4072
+F 0 "D6" V 3664 3992 50  0000 R CNN
+F 1 "BAR42FILM" V 3573 3992 50  0000 R CNN
+F 2 "Package_TO_SOT_SMD:SOT-23" H 3618 3897 50  0001 C CNN
+F 3 "www.st.com/resource/en/datasheet/bar42.pdf" H 3618 4072 50  0001 C CNN
+	1    3618 4072
+	0    -1   -1   0
+$EndComp
+$Comp
+L Device:C C1
+U 1 1 5F143C67
+P 3376 3972
+F 0 "C1" H 3491 4018 50  0000 L CNN
+F 1 "100n" H 3491 3927 50  0000 L CNN
+F 2 "Capacitor_SMD:C_1206_3216Metric" H 3414 3822 50  0001 C CNN
+F 3 "~" H 3376 3972 50  0001 C CNN
+	1    3376 3972
+	1    0    0    -1
+$EndComp
+Wire Wire Line
+	3620 3736 3620 3822
+Wire Wire Line
+	3620 3922 3618 3922
+Wire Wire Line
+	3358 3822 3376 3822
+Connection ~ 3620 3822
+Wire Wire Line
+	3620 3822 3620 3922
+Wire Wire Line
+	2538 3440 2758 3440
+Wire Wire Line
+	2758 3822 2758 3440
+Connection ~ 2758 3440
+Wire Wire Line
+	2758 3440 3260 3440
+Connection ~ 3376 3822
+Wire Wire Line
+	3376 3822 3620 3822
+Wire Wire Line
+	3618 4440 3640 4440
+$Comp
+L power:+3.3V #PWR06
+U 1 1 5DBE0E51
+P 2636 4096
+F 0 "#PWR06" H 2636 3946 50  0001 C CNN
+F 1 "+3.3V" V 2651 4224 50  0000 L CNN
+F 2 "" H 2636 4096 50  0001 C CNN
+F 3 "" H 2636 4096 50  0001 C CNN
+	1    2636 4096
+	1    0    0    -1
+$EndComp
+Wire Wire Line
+	2978 4100 2636 4100
+Wire Wire Line
+	2636 4100 2636 4096
+$Comp
+L Device:R R6
+U 1 1 5DBEC0DF
+P 2810 4600
+F 0 "R6" V 2603 4600 50  0000 C CNN
+F 1 "680" V 2694 4600 50  0000 C CNN
+F 2 "Resistor_SMD:R_1206_3216Metric" V 2740 4600 50  0001 C CNN
+F 3 "~" H 2810 4600 50  0001 C CNN
+	1    2810 4600
+	0    1    1    0
+$EndComp
+$Comp
+L Device:R R5
+U 1 1 5F19E15B
+P 2636 4250
+F 0 "R5" H 2706 4296 50  0000 L CNN
+F 1 "2k" H 2706 4205 50  0000 L CNN
+F 2 "Resistor_SMD:R_1206_3216Metric" V 2566 4250 50  0001 C CNN
+F 3 "~" H 2636 4250 50  0001 C CNN
+	1    2636 4250
+	1    0    0    -1
+$EndComp
+Connection ~ 2636 4100
+Wire Wire Line
+	2518 4460 2636 4460
+Wire Wire Line
+	2636 4460 2636 4400
+Wire Wire Line
+	2636 4460 3618 4460
+Wire Wire Line
+	3618 4222 3618 4440
+Connection ~ 2636 4460
+Connection ~ 3618 4440
+Wire Wire Line
+	3618 4440 3618 4460
+Wire Wire Line
+	2960 4600 2978 4600
+Wire Wire Line
+	2978 4600 2978 4400
+Wire Wire Line
+	2978 4600 2978 4640
+Wire Wire Line
+	2978 4640 3020 4640
+Connection ~ 2978 4600
+Wire Wire Line
+	2660 4600 2520 4600
+$Comp
+L Diode:BAR42FILM D4
+U 1 1 5F1B960F
+P 2908 3822
+F 0 "D4" H 2908 3605 50  0000 C CNN
+F 1 "BAR42FILM" H 2908 3696 50  0000 C CNN
+F 2 "Package_TO_SOT_SMD:SOT-23" H 2908 3647 50  0001 C CNN
+F 3 "www.st.com/resource/en/datasheet/bar42.pdf" H 2908 3822 50  0001 C CNN
+	1    2908 3822
+	-1   0    0    1
+$EndComp
+Connection ~ 4315 2150
+$Comp
 L Diode:1N4148WS D7
 U 1 1 5F1E8679
@@
 	0    -1   -1   0
 $EndComp
-$Comp
-L Diode:1N4148WS D8
-U 1 1 5F1F6AFD
-P 4315 2300
-F 0 "D8" V 4361 2220 50  0000 R CNN
-F 1 "1N4148WS" V 4270 2220 50  0000 R CNN
-F 2 "Diode_SMD:D_SOD-323" H 4315 2125 50  0001 C CNN
-F 3 "https://www.vishay.com/docs/85751/1n4148ws.pdf" H 4315 2300 50  0001 C CNN
-	1    4315 2300
-	0    -1   -1   0
-$EndComp
-Connection ~ 4315 2150
-Wire Wire Line
-	4315 2450 4315 2470
-Wire Wire Line
-	4315 2470 4660 2470
-Wire Wire Line
-	4660 2470 4660 2480
-Connection ~ 4315 2470
-Wire Wire Line
-	4315 2470 4315 2490
-$Comp
-L Diode:BAR42FILM D5
-U 1 1 5F0E2174
-P 3410 3442
-F 0 "D5" H 3410 3723 50  0000 C CNN
-F 1 "BAR42FILM" H 3410 3632 50  0000 C CNN
-F 2 "Package_TO_SOT_SMD:SOT-23" H 3410 3267 50  0001 C CNN
-F 3 "www.st.com/resource/en/datasheet/bar42.pdf" H 3410 3442 50  0001 C CNN
-	1    3410 3442
-	1    0    0    -1
-$EndComp
-Text GLabel 3836 3438 2    50   Input ~ 0
-EN
-Wire Wire Line
-	3834 3436 3836 3438
-Wire Wire Line
-	2480 3440 2538 3440
-Wire Wire Line
-	3260 3440 3260 3442
-Connection ~ 2538 3440
-Wire Wire Line
-	3572 3436 3572 3442
-Wire Wire Line
-	3572 3442 3560 3442
-Wire Wire Line
-	3620 3436 3834 3436
-Wire Wire Line
-	3572 3436 3620 3436
-Connection ~ 3620 3436
-$Comp
-L Device:R R9
-U 1 1 5DBEDE1B
-P 3620 3586
-F 0 "R9" H 3550 3540 50  0000 R CNN
-F 1 "2k" H 3550 3631 50  0000 R CNN
-F 2 "Resistor_SMD:R_1206_3216Metric" V 3550 3586 50  0001 C CNN
-F 3 "~" H 3620 3586 50  0001 C CNN
-	1    3620 3586
-	-1   0    0    1
-$EndComp
-$Comp
-L Diode:BAR42FILM D6
-U 1 1 5F139EE6
-P 3618 4072
-F 0 "D6" V 3664 3992 50  0000 R CNN
-F 1 "BAR42FILM" V 3573 3992 50  0000 R CNN
-F 2 "Package_TO_SOT_SMD:SOT-23" H 3618 3897 50  0001 C CNN
-F 3 "www.st.com/resource/en/datasheet/bar42.pdf" H 3618 4072 50  0001 C CNN
-	1    3618 4072
-	0    -1   -1   0
-$EndComp
-$Comp
-L Device:C C1
-U 1 1 5F143C67
-P 3376 3972
-F 0 "C1" H 3491 4018 50  0000 L CNN
-F 1 "100n" H 3491 3927 50  0000 L CNN
-F 2 "Capacitor_SMD:C_1206_3216Metric" H 3414 3822 50  0001 C CNN
-F 3 "~" H 3376 3972 50  0001 C CNN
-	1    3376 3972
-	1    0    0    -1
-$EndComp
-Wire Wire Line
-	3620 3736 3620 3822
-Wire Wire Line
-	3620 3922 3618 3922
-Wire Wire Line
-	3358 3822 3376 3822
-Connection ~ 3620 3822
-Wire Wire Line
-	3620 3822 3620 3922
-Wire Wire Line
-	2538 3440 2758 3440
-Wire Wire Line
-	2758 3822 2758 3440
-Connection ~ 2758 3440
-Wire Wire Line
-	2758 3440 3260 3440
-Connection ~ 3376 3822
-Wire Wire Line
-	3376 3822 3620 3822
-Wire Wire Line
-	3618 4440 3640 4440
-$Comp
-L power:+3.3V #PWR06
-U 1 1 5DBE0E51
-P 2636 4096
-F 0 "#PWR06" H 2636 3946 50  0001 C CNN
-F 1 "+3.3V" V 2651 4224 50  0000 L CNN
-F 2 "" H 2636 4096 50  0001 C CNN
-F 3 "" H 2636 4096 50  0001 C CNN
-	1    2636 4096
-	1    0    0    -1
-$EndComp
-Wire Wire Line
-	2978 4100 2636 4100
-Wire Wire Line
-	2636 4100 2636 4096
-$Comp
-L Device:R R6
-U 1 1 5DBEC0DF
-P 2810 4600
-F 0 "R6" V 2603 4600 50  0000 C CNN
-F 1 "680" V 2694 4600 50  0000 C CNN
-F 2 "Resistor_SMD:R_1206_3216Metric" V 2740 4600 50  0001 C CNN
-F 3 "~" H 2810 4600 50  0001 C CNN
-	1    2810 4600
-	0    1    1    0
-$EndComp
-$Comp
-L Device:R R5
-U 1 1 5F19E15B
-P 2636 4250
-F 0 "R5" H 2706 4296 50  0000 L CNN
-F 1 "2k" H 2706 4205 50  0000 L CNN
-F 2 "Resistor_SMD:R_1206_3216Metric" V 2566 4250 50  0001 C CNN
-F 3 "~" H 2636 4250 50  0001 C CNN
-	1    2636 4250
-	1    0    0    -1
-$EndComp
-Connection ~ 2636 4100
-Wire Wire Line
-	2518 4460 2636 4460
-Wire Wire Line
-	2636 4460 2636 4400
-Wire Wire Line
-	2636 4460 3618 4460
-Wire Wire Line
-	3618 4222 3618 4440
-Connection ~ 2636 4460
-Connection ~ 3618 4440
-Wire Wire Line
-	3618 4440 3618 4460
-Wire Wire Line
-	2960 4600 2978 4600
-Wire Wire Line
-	2978 4600 2978 4400
-Wire Wire Line
-	2978 4600 2978 4640
-Wire Wire Line
-	2978 4640 3020 4640
-Connection ~ 2978 4600
-Wire Wire Line
-	2660 4600 2520 4600
-$Comp
-L Diode:BAR42FILM D4
-U 1 1 5F1B960F
-P 2908 3822
-F 0 "D4" H 2908 3605 50  0000 C CNN
-F 1 "BAR42FILM" H 2908 3696 50  0000 C CNN
-F 2 "Package_TO_SOT_SMD:SOT-23" H 2908 3647 50  0001 C CNN
-F 3 "www.st.com/resource/en/datasheet/bar42.pdf" H 2908 3822 50  0001 C CNN
-	1    2908 3822
-	-1   0    0    1
-$EndComp
 $EndSCHEMATC
