File: kicad/sboxnet-booster/sboxnet-booster.sch (KiCad schematic (older format))
At the start: 67 parts, among them J1 sboxnet-stecker_02x17, J3 Conn_01x02_Male, J4 Conn_01x02_Male, J5 Screw_Terminal_01x04, J6 Screw_Terminal_01x04, J7 Power von externen 15V/4A Net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, SW1 Öffner, U1 L6206PSO-sboxnet, U2 L78L12_SOT89, U3 SN65HVD230

Commit message: fixed booster schema
Changed lines of the file:
@@
 	2250 2850 2250 2800
 Wire Wire Line
-	1569 4840 1850 4840
+	1569 4840 1820 4840
 Wire Wire Line
-	1030 4940 1069 4940
+	1030 4940 1050 4940
 Wire Wire Line
-	1030 4840 1069 4840
+	1030 4840 1050 4840
 $Comp
 L power:PWR_FLAG #FLG0101
@@
 Wire Wire Line
 	1760 3939 1760 3940
+$Comp
+L power:PWR_FLAG #FLG0102
+U 1 1 5F559ADC
+P 1050 4840
+F 0 "#FLG0102" H 1050 4915 50  0001 C CNN
+F 1 "PWR_FLAG" H 1050 5013 50  0000 C CNN
+F 2 "" H 1050 4840 50  0001 C CNN
+F 3 "~" H 1050 4840 50  0001 C CNN
+	1    1050 4840
+	1    0    0    -1
+$EndComp
+Connection ~ 1050 4840
 Wire Wire Line
-	2250 2260 2250 2300
+	1050 4840 1069 4840
+$Comp
+L power:PWR_FLAG #FLG0103
+U 1 1 5F55AFE9
+P 1820 4840
+F 0 "#FLG0103" H 1820 4915 50  0001 C CNN
+F 1 "PWR_FLAG" H 1820 5013 50  0000 C CNN
+F 2 "" H 1820 4840 50  0001 C CNN
+F 3 "~" H 1820 4840 50  0001 C CNN
+	1    1820 4840
+	1    0    0    -1
+$EndComp
+Connection ~ 1820 4840
+Wire Wire Line
+	1820 4840 1850 4840
+$Comp
+L power:PWR_FLAG #FLG0104
+U 1 1 5F55C2A6
+P 1050 4940
+F 0 "#FLG0104" H 1050 5015 50  0001 C CNN
+F 1 "PWR_FLAG" H 1050 5113 50  0000 C CNN
+F 2 "" H 1050 4940 50  0001 C CNN
+F 3 "~" H 1050 4940 50  0001 C CNN
+	1    1050 4940
+	-1   0    0    1
+$EndComp
+Connection ~ 1050 4940
+Wire Wire Line
+	1050 4940 1069 4940
 $EndSCHEMATC

Commit message: new booster 20200927
Other:
- note added: "ON"
- note added: "OV"
- note removed: "OVERCURRENT"
Changed lines of the file:
@@
 	0    -1   -1   0
 $EndComp
-Text Notes 2265 1270 2    50   ~ 0
+Text Notes 1920 830  3    50   ~ 0
 NOTAUS
 Text Notes 2225 1470 2    50   ~ 0
@@
 	0    -1   -1   0
 $EndComp
-Text Notes 1755 1210 3    50   ~ 0
-OVERCURRENT
+Text Notes 1430 780  3    50   ~ 0
+OV
 Text Notes 1680 1470 2    50   ~ 0
 ge
@@
 	0    -1   -1   0
 $EndComp
-Text Notes 1200 1350 3    50   ~ 0
+Text Notes 840  720  3    50   ~ 0
 Abschaltung
 Text Notes 1135 1450 2    50   ~ 0
@@
 Wire Wire Line
 	1050 4940 1069 4940
+Text Notes 2410 840  3    50   ~ 0
+ON
 $EndSCHEMATC
