File: kicad/sboxnet-gbm/sboxnet-gbm.kicad_pcb (KiCad board)
At the start: 2 copper layers, 102.4 x 85.1 mm, 46 parts, among them J1 Screw_Terminal_01x04, J2 Screw_Terminal_01x04, J3 Screw_Terminal_01x04, J4 sboxnet-stecker_02x17, J5 Screw_Terminal_01x04, U1 LTV-844, U2 LTV-844, U3 LTV-844, U4 SN65HVD230

Commit message: booster DCC Input
Parts:
- added TP1: TestPoint, Connector_PinHeader_2.54mm:PinHeader_1x01_P2.54mm_Vertical, F.Cu at (62.0, 54.6)
Routing:
- net PA0: track 27.3 -> 29.4 mm
